Commit message: Migrated all plugins to rosflight_plugins package
Also moved all parameters to yaml file, rather than using sdf param server.

File: rosplane_sim/agents/default_fixedwing/default_fixedwing.xacro (robot description, xacro)
@@ -62,44 +62,36 @@
   <xacro:aircraft_truth
     namespace="${namespace}"
-    parent_link="${namespace}/base_link"
-    wind_speed_topic="gazebo/wind_speed"/>
+    parent_link="${namespace}/base_link"/>
   <!-- Aerodynamics -->
   <xacro:include filename="$(find rosplane_sim)/xacro/aircraft_forces_and_moments.xacro"/>
-  <xacro:myTwinDream
+  <xacro:aircraft_dynamics
     namespace="${namespace}"
-    parent_link="${namespace}/base_link"
-    command_topic="command"/>
+    parent_link="${namespace}/base_link"/>
   <!-- GPS -->
-  <!-- <xacro:include filename="$(find fcu_sim_plugins)/xacro/GPS.xacro"/>
-  <xacro:GPS_BYU
+  <xacro:include filename="$(find rosflight_plugins)/xacro/GPS.xacro"/>
+  <xacro:gps_plugin_macro
     namespace="${namespace}"
-    parent_link="${namespace}/base_link"
-    GPS_topic="gps/data"
-    update_rate="1">
-  </xacro:GPS_BYU> -->
+    parent_link="${namespace}/base_link">
+  </xacro:gps_plugin_macro>
   <!-- IMU -->
-  <!-- <xacro:include filename="$(find fcu_sim_plugins)/xacro/imu.xacro"/>
-  <xacro:IMU_MPU6050
+  <xacro:include filename="$(find rosflight_plugins)/xacro/imu.xacro"/>
+  <xacro:imu_plugin_macro
     namespace="${namespace}"
-    parent_link="${namespace}/base_link"
-    imu_topic="imu/data"
-    update_rate="500">
-  </xacro:IMU_MPU6050> -->
+    parent_link="${namespace}/base_link">
+  </xacro:imu_plugin_macro>
   <!-- Airspeed -->
-  <!-- <xacro:include filename="$(find fcu_sim_plugins)/xacro/airspeed.xacro"/>
-  <xacro:airspeed_MPXV5004G
+  <xacro:include filename="$(find rosflight_plugins)/xacro/airspeed.xacro"/>
+  <xacro:airspeed_plugin_macro
     namespace="${namespace}"
-    parent_link="${namespace}/base_link"
-    airspeed_topic="airspeed/data">
-  </xacro:airspeed_MPXV5004G> -->
+    parent_link="${namespace}/base_link">
+  </xacro:airspeed_plugin_macro>
   <!-- Barometer -->
-  <!-- <xacro:include filename="$(find fcu_sim_plugins)/xacro/barometer.xacro"/>
-  <xacro:Barometer_MS5611
+  <xacro:include filename="$(find rosflight_plugins)/xacro/barometer.xacro"/>
+  <xacro:barometer_plugin_macro
     namespace="${namespace}"
-    parent_link="${namespace}/base_link"
-    baro_topic="baro/data">
-  </xacro:Barometer_MS5611> -->
+    parent_link="${namespace}/base_link">
+  </xacro:barometer_plugin_macro>
   <!-- Chase Camera -->
-  <xacro:include filename="$(find fcu_sim_plugins)/xacro/camera.xacro"/>
+  <!-- <xacro:include filename="$(find fcu_sim_plugins)/xacro/camera.xacro"/>
   <xacro:simple_camera
     namespace="${namespace}/chase"
@@ -110,5 +102,5 @@
     image_camera_info_topic="camera_info">
     <origin xyz="-${1.1*body_length} 0 ${0.8*body_height}"/>
-  </xacro:simple_camera>
+  </xacro:simple_camera> -->
   <!-- Gimbal -->
   <!-- <xacro:include filename="$(find fcu_sim_plugins)/xacro/gimbal.xacro"/>
@@ -123,11 +115,3 @@
     <origin xyz="-${0.4*body_length} 0 -${0.4*body_height}" rpy="0 0 0"/>
   </xacro:gimbal_ZENMUSE> -->
-  <!-- Sonar -->
-  <!-- <xacro:include filename="$(find fcu_sim_plugins)/xacro/sonar.xacro"/>
-  <xacro:Sonar_MB1030
-    namespace="${namespace}"
-    parent_link="${namespace}/base_link"
-    sonar_topic="sonar/data">
-    <origin xyz="0 0 0" rpy="0 0 0"/>
-  </xacro:Sonar_MB1030> -->
 </robot>
